File: projects/crow-audio-carrier-v1/03_tscircuit/kicad/crow_audio_carrier_v1.kicad_sch (KiCad schematic)
At the start: 333 parts, among them J1 615008160221, J10 TMM-106-01-L-D, J11 TMM-106-01-L-D, J2 615008160221, J3 615008160221, J4 615008160221, J5 615008160221, J6 615008160221, J7 615008160221, J8 615008160221, J9 43650-0200

Commit message: release(crow): qualify all-SMD carrier assembly
Parts:
- C_FILT1_470U, C_FILT2_470U, C_HOLD1, C_HOLD2: Supplier Part Numbers {"jlcpcb": []} -> {"jlcpcb": ["C178530"]}
- F_IN: Supplier Part Numbers {"jlcpcb": []} -> {"jlcpcb": ["C22870534"]}
- U_ADC: Supplier Part Numbers {"jlcpcb": []} -> {"jlcpcb": ["C42457798"]}
