File: projects/crow-usb-carrier-v1/04_kicad/crow_carrier.kicad_sch (KiCad schematic)
At the start: 493 parts, among them J1 615008160221, J2 615008160221, J3 615008160221, J4 615008160221, J5 615008160221, J6 615008160221, J7 615008160221, J8 615008160221

Commit message: Regenerate Crow schematic and record exact remaining admission checks
Parts:
- removed C_DUMP_TIME: 15nF, Capacitor_SMD:C_0805_2012Metric, symbol elt:SYM_C_DUMP_TIME
- removed C_FILT1_10U: 10uF, Capacitor_SMD:C_0805_2012Metric, symbol elt:SYM_C_FILT1_10U
- removed C_FILT1_1U: 1uF, Capacitor_SMD:C_0603_1608Metric, symbol elt:SYM_C_FILT1_1U
- removed C_FILT1_470U: 470uF, crow_usb_analog:Panasonic_EEEFK1A471P_8x10.2_Exact, symbol elt:SYM_C_FILT1_470U
- removed C_FILT2_10U: 10uF, Capacitor_SMD:C_0805_2012Metric, symbol elt:SYM_C_FILT2_10U
- removed C_FILT2_1U: 1uF, Capacitor_SMD:C_0603_1608Metric, symbol elt:SYM_C_FILT2_1U
- removed C_FILT2_470U: 470uF, crow_usb_analog:Panasonic_EEEFK1A471P_8x10.2_Exact, symbol elt:SYM_C_FILT2_470U
- removed C_LDO_A: 4.7uF, Capacitor_SMD:C_0805_2012Metric, symbol elt:SYM_C_LDO_A
- removed C_LDO_D: 4.7uF, Capacitor_SMD:C_0805_2012Metric, symbol elt:SYM_C_LDO_D
- removed C_MCLK_BUF: 100nF, Capacitor_SMD:C_0402_1005Metric, symbol elt:SYM_C_MCLK_BUF
- removed C_U_1V8_OUT_2: 47uF, crow_usb_power_aux:TDK_CKG57K_JLead, symbol elt:SYM_C_U_1V8_OUT_2
- removed C_U_3V3X_OUT_2: 47uF, crow_usb_power_aux:TDK_CKG57K_JLead, symbol elt:SYM_C_U_3V3X_OUT_2
- removed C_U_CORE_OUT_2: 47uF, crow_usb_power_aux:TDK_CKG57K_JLead, symbol elt:SYM_C_U_CORE_OUT_2
- removed C_VDDA1_10N: 10nF, Capacitor_SMD:C_0402_1005Metric, symbol elt:SYM_C_VDDA1_10N
- removed C_VDDA1_4U7: 4.7uF, Capacitor_SMD:C_0603_1608Metric, symbol elt:SYM_C_VDDA1_4U7
- removed C_VDDA2_10N: 10nF, Capacitor_SMD:C_0402_1005Metric, symbol elt:SYM_C_VDDA2_10N
- removed C_VDDA2_4U7: 4.7uF, Capacitor_SMD:C_0603_1608Metric, symbol elt:SYM_C_VDDA2_4U7
- removed C_VDDIO: 100nF, Capacitor_SMD:C_0402_1005Metric, symbol elt:SYM_C_VDDIO
- removed C_VMID1_470N: 470nF, Capacitor_SMD:C_0603_1608Metric, symbol elt:SYM_C_VMID1_470N
- removed C_VMID1_4U7: 10uF, Capacitor_SMD:C_0805_2012Metric, symbol elt:SYM_C_VMID1_4U7
- removed C_VMID2_470N: 470nF, Capacitor_SMD:C_0603_1608Metric, symbol elt:SYM_C_VMID2_470N
- removed C_VMID2_4U7: 10uF, Capacitor_SMD:C_0805_2012Metric, symbol elt:SYM_C_VMID2_4U7
- removed Q_MCLK_GATE: AO3400A, Package_TO_SOT_SMD:SOT-23, symbol elt:SYM_Q_MCLK_GATE
- removed R_CFG1: 4.7kΩ, Resistor_SMD:R_0402_1005Metric, symbol elt:SYM_R_CFG1
- removed R_CFG2: 0Ω, Resistor_SMD:R_0402_1005Metric, symbol elt:SYM_R_CFG2
- removed R_CFG4: 4.7kΩ, Resistor_SMD:R_0402_1005Metric, symbol elt:SYM_R_CFG4
- removed R_CFG5: 100kΩ, Resistor_SMD:R_0402_1005Metric, symbol elt:SYM_R_CFG5
- removed R_FILT1P: 1Ω, Resistor_SMD:R_1206_3216Metric, symbol elt:SYM_R_FILT1P
- removed R_FILT2P: 1Ω, Resistor_SMD:R_1206_3216Metric, symbol elt:SYM_R_FILT2P
- removed R_MCLK: 33Ω, Resistor_SMD:R_0402_1005Metric, symbol elt:SYM_R_MCLK
- removed R_MCLK_OE_PU: 10kΩ, Resistor_SMD:R_0402_1005Metric, symbol elt:SYM_R_MCLK_OE_PU
- removed R_MCLK_RAW_PD: 100kΩ, Resistor_SMD:R_0402_1005Metric, symbol elt:SYM_R_MCLK_RAW_PD
- removed U_ADC: CS5308P-DNR, crow_usb_analog:Cirrus_CS5308P_QFN48_6x6_P0.4_EP4.6, symbol elt:SYM_U_ADC
- removed U_MCLK_BUF: SN74LVC1G125DCKT, crow_usb_digital:TI_DCK0005A_SC70_5, symbol elt:SYM_U_MCLK_BUF
- added C_1V8_FF: 120pF, Capacitor_SMD:C_0402_1005Metric, symbol elt:SYM_C_1V8_FF
- added C_3V3X_FF: 120pF, Capacitor_SMD:C_0402_1005Metric, symbol elt:SYM_C_3V3X_FF
- added C_ADC_AC1N1: 47uF, crow_usb_power_aux:Murata_GRM32E_1210, symbol elt:SYM_C_ADC_AC1N1
- added C_ADC_AC1N2: 47uF, crow_usb_power_aux:Murata_GRM32E_1210, symbol elt:SYM_C_ADC_AC1N2
- added C_ADC_AC1P1: 47uF, crow_usb_power_aux:Murata_GRM32E_1210, symbol elt:SYM_C_ADC_AC1P1
- added C_ADC_AC1P2: 47uF, crow_usb_power_aux:Murata_GRM32E_1210, symbol elt:SYM_C_ADC_AC1P2
- added C_ADC_AC2N1: 47uF, crow_usb_power_aux:Murata_GRM32E_1210, symbol elt:SYM_C_ADC_AC2N1
- added C_ADC_AC2N2: 47uF, crow_usb_power_aux:Murata_GRM32E_1210, symbol elt:SYM_C_ADC_AC2N2
- added C_ADC_AC2P1: 47uF, crow_usb_power_aux:Murata_GRM32E_1210, symbol elt:SYM_C_ADC_AC2P1
- added C_ADC_AC2P2: 47uF, crow_usb_power_aux:Murata_GRM32E_1210, symbol elt:SYM_C_ADC_AC2P2
- added C_ADC_AC3N1: 47uF, crow_usb_power_aux:Murata_GRM32E_1210, symbol elt:SYM_C_ADC_AC3N1
- added C_ADC_AC3N2: 47uF, crow_usb_power_aux:Murata_GRM32E_1210, symbol elt:SYM_C_ADC_AC3N2
- added C_ADC_AC3P1: 47uF, crow_usb_power_aux:Murata_GRM32E_1210, symbol elt:SYM_C_ADC_AC3P1
- added C_ADC_AC3P2: 47uF, crow_usb_power_aux:Murata_GRM32E_1210, symbol elt:SYM_C_ADC_AC3P2
- added C_ADC_AC4N1: 47uF, crow_usb_power_aux:Murata_GRM32E_1210, symbol elt:SYM_C_ADC_AC4N1
- added C_ADC_AC4N2: 47uF, crow_usb_power_aux:Murata_GRM32E_1210, symbol elt:SYM_C_ADC_AC4N2
- added C_ADC_AC4P1: 47uF, crow_usb_power_aux:Murata_GRM32E_1210, symbol elt:SYM_C_ADC_AC4P1
- added C_ADC_AC4P2: 47uF, crow_usb_power_aux:Murata_GRM32E_1210, symbol elt:SYM_C_ADC_AC4P2
- added C_ADC_AC5N1: 47uF, crow_usb_power_aux:Murata_GRM32E_1210, symbol elt:SYM_C_ADC_AC5N1
- added C_ADC_AC5N2: 47uF, crow_usb_power_aux:Murata_GRM32E_1210, symbol elt:SYM_C_ADC_AC5N2
- added C_ADC_AC5P1: 47uF, crow_usb_power_aux:Murata_GRM32E_1210, symbol elt:SYM_C_ADC_AC5P1
- added C_ADC_AC5P2: 47uF, crow_usb_power_aux:Murata_GRM32E_1210, symbol elt:SYM_C_ADC_AC5P2
- added C_ADC_AC6N1: 47uF, crow_usb_power_aux:Murata_GRM32E_1210, symbol elt:SYM_C_ADC_AC6N1
- added C_ADC_AC6N2: 47uF, crow_usb_power_aux:Murata_GRM32E_1210, symbol elt:SYM_C_ADC_AC6N2
- added C_ADC_AC6P1: 47uF, crow_usb_power_aux:Murata_GRM32E_1210, symbol elt:SYM_C_ADC_AC6P1
- added C_ADC_AC6P2: 47uF, crow_usb_power_aux:Murata_GRM32E_1210, symbol elt:SYM_C_ADC_AC6P2
- added C_ADC_AC7N1: 47uF, crow_usb_power_aux:Murata_GRM32E_1210, symbol elt:SYM_C_ADC_AC7N1
- added C_ADC_AC7N2: 47uF, crow_usb_power_aux:Murata_GRM32E_1210, symbol elt:SYM_C_ADC_AC7N2
- added C_ADC_AC7P1: 47uF, crow_usb_power_aux:Murata_GRM32E_1210, symbol elt:SYM_C_ADC_AC7P1
- added C_ADC_AC7P2: 47uF, crow_usb_power_aux:Murata_GRM32E_1210, symbol elt:SYM_C_ADC_AC7P2
- added C_ADC_AC8N1: 47uF, crow_usb_power_aux:Murata_GRM32E_1210, symbol elt:SYM_C_ADC_AC8N1
- added C_ADC_AC8N2: 47uF, crow_usb_power_aux:Murata_GRM32E_1210, symbol elt:SYM_C_ADC_AC8N2
- added C_ADC_AC8P1: 47uF, crow_usb_power_aux:Murata_GRM32E_1210, symbol elt:SYM_C_ADC_AC8P1
- added C_ADC_AC8P2: 47uF, crow_usb_power_aux:Murata_GRM32E_1210, symbol elt:SYM_C_ADC_AC8P2
- added C_ADC_A_AREG_100N: 100nF, Capacitor_SMD:C_0402_1005Metric, symbol elt:SYM_C_ADC_A_AREG_100N
- added C_ADC_A_AREG_1U: 1uF, Capacitor_SMD:C_0603_1608Metric, symbol elt:SYM_C_ADC_A_AREG_1U
- added C_ADC_A_AVDD_100N: 100nF, Capacitor_SMD:C_0402_1005Metric, symbol elt:SYM_C_ADC_A_AVDD_100N
- added C_ADC_A_AVDD_10U: 10uF, Capacitor_SMD:C_0805_2012Metric, symbol elt:SYM_C_ADC_A_AVDD_10U
- added C_ADC_A_DREG_100N: 100nF, Capacitor_SMD:C_0402_1005Metric, symbol elt:SYM_C_ADC_A_DREG_100N
- added C_ADC_A_DREG_1U: 1uF, Capacitor_SMD:C_0603_1608Metric, symbol elt:SYM_C_ADC_A_DREG_1U
- added C_ADC_A_IOVDD_100N: 100nF, Capacitor_SMD:C_0402_1005Metric, symbol elt:SYM_C_ADC_A_IOVDD_100N
- added C_ADC_A_IOVDD_10U: 10uF, Capacitor_SMD:C_0805_2012Metric, symbol elt:SYM_C_ADC_A_IOVDD_10U
- added C_ADC_A_VREF_100N: 100nF, Capacitor_SMD:C_0402_1005Metric, symbol elt:SYM_C_ADC_A_VREF_100N
- added C_ADC_A_VREF_10U: 10uF, Capacitor_SMD:C_0805_2012Metric, symbol elt:SYM_C_ADC_A_VREF_10U
- added C_ADC_B_AREG_100N: 100nF, Capacitor_SMD:C_0402_1005Metric, symbol elt:SYM_C_ADC_B_AREG_100N
- added C_ADC_B_AREG_1U: 1uF, Capacitor_SMD:C_0603_1608Metric, symbol elt:SYM_C_ADC_B_AREG_1U
- added C_ADC_B_AVDD_100N: 100nF, Capacitor_SMD:C_0402_1005Metric, symbol elt:SYM_C_ADC_B_AVDD_100N
- added C_ADC_B_AVDD_10U: 10uF, Capacitor_SMD:C_0805_2012Metric, symbol elt:SYM_C_ADC_B_AVDD_10U
- added C_ADC_B_DREG_100N: 100nF, Capacitor_SMD:C_0402_1005Metric, symbol elt:SYM_C_ADC_B_DREG_100N
- added C_ADC_B_DREG_1U: 1uF, Capacitor_SMD:C_0603_1608Metric, symbol elt:SYM_C_ADC_B_DREG_1U
- added C_ADC_B_IOVDD_100N: 100nF, Capacitor_SMD:C_0402_1005Metric, symbol elt:SYM_C_ADC_B_IOVDD_100N
- added C_ADC_B_IOVDD_10U: 10uF, Capacitor_SMD:C_0805_2012Metric, symbol elt:SYM_C_ADC_B_IOVDD_10U
- added C_ADC_B_VREF_100N: 100nF, Capacitor_SMD:C_0402_1005Metric, symbol elt:SYM_C_ADC_B_VREF_100N
- added C_ADC_B_VREF_10U: 10uF, Capacitor_SMD:C_0805_2012Metric, symbol elt:SYM_C_ADC_B_VREF_10U
- added C_ADC_I2C_A: 100nF, Capacitor_SMD:C_0402_1005Metric, symbol elt:SYM_C_ADC_I2C_A
- added C_ADC_I2C_B: 100nF, Capacitor_SMD:C_0402_1005Metric, symbol elt:SYM_C_ADC_I2C_B
- added C_ADC_PWR_BAD: 100nF, Capacitor_SMD:C_0402_1005Metric, symbol elt:SYM_C_ADC_PWR_BAD
- added C_CORE_FF: 120pF, Capacitor_SMD:C_0402_1005Metric, symbol elt:SYM_C_CORE_FF
- added C_DUMP_TIME1: 15nF, Capacitor_SMD:C_0805_2012Metric, symbol elt:SYM_C_DUMP_TIME1
- added C_DUMP_TIME2: 15nF, Capacitor_SMD:C_0805_2012Metric, symbol elt:SYM_C_DUMP_TIME2
- added C_DUMP_TIME3: 15nF, Capacitor_SMD:C_0805_2012Metric, symbol elt:SYM_C_DUMP_TIME3
- added C_DUMP_TIME4: 15nF, Capacitor_SMD:C_0805_2012Metric, symbol elt:SYM_C_DUMP_TIME4
- added C_DUMP_TIME5: 15nF, Capacitor_SMD:C_0805_2012Metric, symbol elt:SYM_C_DUMP_TIME5
- added C_DUMP_TIME6: 15nF, Capacitor_SMD:C_0805_2012Metric, symbol elt:SYM_C_DUMP_TIME6
- added C_DUMP_TIME7: 15nF, Capacitor_SMD:C_0805_2012Metric, symbol elt:SYM_C_DUMP_TIME7
- added C_DUMP_TIME8: 15nF, Capacitor_SMD:C_0805_2012Metric, symbol elt:SYM_C_DUMP_TIME8
- added C_HOLD10: 470uF, crow_usb_analog:Panasonic_EEEFK1A471P_8x10.2_Exact, symbol elt:SYM_C_HOLD10
- added C_HOLD11: 470uF, crow_usb_analog:Panasonic_EEEFK1A471P_8x10.2_Exact, symbol elt:SYM_C_HOLD11
- added C_HOLD12: 470uF, crow_usb_analog:Panasonic_EEEFK1A471P_8x10.2_Exact, symbol elt:SYM_C_HOLD12
- added C_HOLD13: 470uF, crow_usb_analog:Panasonic_EEEFK1A471P_8x10.2_Exact, symbol elt:SYM_C_HOLD13
- added C_HOLD14: 470uF, crow_usb_analog:Panasonic_EEEFK1A471P_8x10.2_Exact, symbol elt:SYM_C_HOLD14
- added C_HOLD15: 470uF, crow_usb_analog:Panasonic_EEEFK1A471P_8x10.2_Exact, symbol elt:SYM_C_HOLD15
- added C_HOLD16: 470uF, crow_usb_analog:Panasonic_EEEFK1A471P_8x10.2_Exact, symbol elt:SYM_C_HOLD16
- added C_HOLD3: 470uF, crow_usb_analog:Panasonic_EEEFK1A471P_8x10.2_Exact, symbol elt:SYM_C_HOLD3
- added C_HOLD4: 470uF, crow_usb_analog:Panasonic_EEEFK1A471P_8x10.2_Exact, symbol elt:SYM_C_HOLD4
- added C_HOLD5: 470uF, crow_usb_analog:Panasonic_EEEFK1A471P_8x10.2_Exact, symbol elt:SYM_C_HOLD5
- added C_HOLD6: 470uF, crow_usb_analog:Panasonic_EEEFK1A471P_8x10.2_Exact, symbol elt:SYM_C_HOLD6
- added C_HOLD7: 470uF, crow_usb_analog:Panasonic_EEEFK1A471P_8x10.2_Exact, symbol elt:SYM_C_HOLD7
- added C_HOLD8: 470uF, crow_usb_analog:Panasonic_EEEFK1A471P_8x10.2_Exact, symbol elt:SYM_C_HOLD8
- added C_HOLD9: 470uF, crow_usb_analog:Panasonic_EEEFK1A471P_8x10.2_Exact, symbol elt:SYM_C_HOLD9
- added C_PWR_CT2: 1uF, Capacitor_SMD:C_0603_1608Metric, symbol elt:SYM_C_PWR_CT2
- added C_PWR_CT3: 1uF, Capacitor_SMD:C_0603_1608Metric, symbol elt:SYM_C_PWR_CT3
- added Q_ADC_PWR_RST: 2N7002K-7, crow_usb_analog:Diodes_2N7002K_SOT23_Exact, symbol elt:SYM_Q_ADC_PWR_RST
- added R_1V8_FB_BOTTOM: 100kΩ, Resistor_SMD:R_0402_1005Metric, symbol elt:SYM_R_1V8_FB_BOTTOM
- added R_1V8_FB_TOP: 210kΩ, Resistor_SMD:R_0402_1005Metric, symbol elt:SYM_R_1V8_FB_TOP
- added R_1V8_OK_BOT: 100kΩ, Resistor_SMD:R_0402_1005Metric, symbol elt:SYM_R_1V8_OK_BOT
- added R_1V8_OK_TOP: 52.3kΩ, Resistor_SMD:R_0402_1005Metric, symbol elt:SYM_R_1V8_OK_TOP
- added R_3V3X_FB_BOTTOM: 100kΩ, Resistor_SMD:R_0603_1608Metric, symbol elt:SYM_R_3V3X_FB_BOTTOM
- added R_3V3X_FB_TOP: 453kΩ, Resistor_SMD:R_0603_1608Metric, symbol elt:SYM_R_3V3X_FB_TOP
- added R_ADC_1V8_OK_BOT: 100kΩ, Resistor_SMD:R_0402_1005Metric, symbol elt:SYM_R_ADC_1V8_OK_BOT
- added R_ADC_1V8_OK_TOP: 52.3kΩ, Resistor_SMD:R_0402_1005Metric, symbol elt:SYM_R_ADC_1V8_OK_TOP
- added R_ADC_3V3X_OK_BOT: 100kΩ, Resistor_SMD:R_0402_1005Metric, symbol elt:SYM_R_ADC_3V3X_OK_BOT
- added R_ADC_3V3X_OK_TOP: 169kΩ, Resistor_SMD:R_0402_1005Metric, symbol elt:SYM_R_ADC_3V3X_OK_TOP
- added R_ADC_I2C_SCL_A_PU: 4.7kΩ, Resistor_SMD:R_0402_1005Metric, symbol elt:SYM_R_ADC_I2C_SCL_A_PU
- added R_ADC_I2C_SCL_B_PU: 4.7kΩ, Resistor_SMD:R_0402_1005Metric, symbol elt:SYM_R_ADC_I2C_SCL_B_PU
- added R_ADC_I2C_SDA_A_PU: 4.7kΩ, Resistor_SMD:R_0402_1005Metric, symbol elt:SYM_R_ADC_I2C_SDA_A_PU
- added R_ADC_I2C_SDA_B_PU: 4.7kΩ, Resistor_SMD:R_0402_1005Metric, symbol elt:SYM_R_ADC_I2C_SDA_B_PU
- added R_ADC_OK_BOT: 100kΩ, Resistor_SMD:R_0402_1005Metric, symbol elt:SYM_R_ADC_OK_BOT
- added R_ADC_OK_TOP: 169kΩ, Resistor_SMD:R_0402_1005Metric, symbol elt:SYM_R_ADC_OK_TOP
- added R_ADC_PWR_BAD_PD: 100kΩ, Resistor_SMD:R_0402_1005Metric, symbol elt:SYM_R_ADC_PWR_BAD_PD
- added R_BUCK_FB_BOTTOM: 10kΩ, Resistor_SMD:R_0402_1005Metric, symbol elt:SYM_R_BUCK_FB_BOTTOM
- added R_BUCK_FB_TOP: 40.2kΩ, Resistor_SMD:R_0402_1005Metric, symbol elt:SYM_R_BUCK_FB_TOP
- added R_DUMP_TIME3: 100kΩ, Resistor_SMD:R_0402_1005Metric, symbol elt:SYM_R_DUMP_TIME3
- added R_XU_3V3_OK_BOT: 100kΩ, Resistor_SMD:R_0402_1005Metric, symbol elt:SYM_R_XU_3V3_OK_BOT
- added R_XU_3V3_OK_TOP: 169kΩ, Resistor_SMD:R_0402_1005Metric, symbol elt:SYM_R_XU_3V3_OK_TOP
- added U_ADC_A: TLV320ADC6140IRTWT, crow_usb_analog:TI_RTW0024A_WQFN24_4x4_EP2.6, symbol elt:SYM_U_ADC_A
- added U_ADC_B: TLV320ADC6140IRTWT, crow_usb_analog:TI_RTW0024A_WQFN24_4x4_EP2.6, symbol elt:SYM_U_ADC_B
- added U_ADC_I2C_XLATE: TCA9406DCUR, crow_usb_digital:TI_TCA9406_DCU0008A_VSSOP8, symbol elt:SYM_U_ADC_I2C_XLATE
- added U_ADC_PWR_BAD: SN74LVC1G04DCKR, crow_usb_digital:TI_DCK0005A_SC70_5, symbol elt:SYM_U_ADC_PWR_BAD
- C_A1N, C_A1P, C_A2N, C_A2P, C_A3N, C_A3P, C_A4N, C_A4P, C_A5N, C_A5P, C_A6N, C_A6P, C_A7N, C_A7P, C_A8N, C_A8P: Supplier Part Numbers {"jlcpcb": ["C3778009"]} -> {"jlcpcb": []}
- C_LDO_IN, C_LDO_OUT_1, C_LDO_OUT_2, C_OPA_BULK, C_OUT1, C_OUT2, C_OUT3, C_U_1V8_OUT_1, C_U_3V3X_OUT_1, C_U_CORE_OUT_1: footprint crow_usb_power_aux:TDK_CKG57K_JLead -> crow_usb_power_aux:Murata_GRM32E_1210; Manufacturer Part Number CKG57KX7R1E476M335JH -> GRM32ER71A476KE15L; Supplier Part Numbers {"jlcpcb": ["C2171626"]} -> {"jlcpcb": ["C84494"]}
- J1, J2, J3, J4, J5, J6, J7, J8: Supplier Part Numbers {"jlcpcb": ["C6461980"]} -> {"jlcpcb": []}
- L_U_1V8, L_U_3V3X, L_U_CORE: value 744373240047 -> XFL4015-471MEC; footprint crow_usb_digital:Wurth_WE-LHMI_744373240047 -> crow_usb_digital:Coilcraft_XFL4015_471MEC; Manufacturer Part Number 744373240047 -> XFL4015-471MEC; Supplier Part Numbers {"jlcpcb": ["C19270343"]} -> {"jlcpcb": ["C18221164"]}
- R_CORE_FB_BOTTOM: value 200kΩ -> 100kΩ; Manufacturer Part Number RT0402BRD07200KL -> RT0402BRD07100KL; Supplier Part Numbers {"jlcpcb": ["C728556"]} -> {"jlcpcb": ["C852472"]}
- R_CORE_FB_TOP: value 100kΩ -> 49.9kΩ; Manufacturer Part Number RT0402BRD07100KL -> RT0402BRD0749K9L; Supplier Part Numbers {"jlcpcb": ["C852472"]} -> {"jlcpcb": ["C852808"]}
- U_1V8: value TPS6282518DMQR -> TPS62825DMQR; Manufacturer Part Number TPS6282518DMQR -> TPS62825DMQR; Supplier Part Numbers {"jlcpcb": ["C2072356"]} -> {"jlcpcb": ["C2650334"]}
- U_1V8_OK, U_ADC_1V8_OK: value TPS389018DSER -> TPS389001DSER; footprint crow_usb_digital:TI_DSE0006A_WSON6 -> crow_usb_analog:TI_DSE0006A_Exact; Manufacturer Part Number TPS389018DSER -> TPS389001DSER; Supplier Part Numbers {"jlcpcb": ["C2066910"]} -> {"jlcpcb": ["C1509297"]}
- U_3V3X: value TPS6282533DMQR -> TPS62825DMQR; Manufacturer Part Number TPS6282533DMQR -> TPS62825DMQR; Supplier Part Numbers {"jlcpcb": ["C3189971"]} -> {"jlcpcb": ["C2650334"]}
- U_ADC_3V3X_OK, U_ADC_OK, U_XU_3V3_OK: value TPS389030DSER -> TPS389001DSER; footprint crow_usb_digital:TI_DSE0006A_WSON6 -> crow_usb_analog:TI_DSE0006A_Exact; Manufacturer Part Number TPS389030DSER -> TPS389001DSER; Supplier Part Numbers {"jlcpcb": ["C2066942"]} -> {"jlcpcb": ["C1509297"]}
- U_AFE1, U_AFE2, U_AFE3, U_AFE4, U_AFE5, U_AFE6, U_AFE7, U_AFE8: value OPA2320AID -> OPA2320AIDR; Manufacturer Part Number OPA2320AID -> OPA2320AIDR; Supplier Part Numbers {"jlcpcb": ["C2861439"]} -> {"jlcpcb": ["C2863402"]}
- U_BUCK: value TPSM63603V5RDHR -> TPSM63603RDHR; footprint crow_usb_power:TPSM63603V5RDHR_RDH0030A -> crow_usb_power:TPSM63603RDHR_RDH0030A; Manufacturer Part Number TPSM63603V5RDHR -> TPSM63603RDHR; Supplier Part Numbers {"jlcpcb": ["C5219330"]} -> {"jlcpcb": ["C5219327"]}
- U_ISO1, U_ISO2, U_ISO3, U_ISO4, U_ISO5, U_ISO6, U_ISO7, U_ISO8: value TMUX2821DSGR -> TMUX4827YBHR; footprint crow_usb_analog:TI_DSG0008A_Exact -> crow_usb_analog:TI_YBH0009_C02_TMUX4827; Manufacturer Part Number TMUX2821DSGR -> TMUX4827YBHR; Supplier Part Numbers {"jlcpcb": ["C53283916"]} -> {"jlcpcb": ["C22428234"]}
- Y_AUDIO: value ASFL1-24.576MHZ-EC-T -> SX5M24.576M20F30TNN; footprint crow_usb_digital:Abracon_ASFL1_5032 -> crow_usb_digital:SCTF_SX5M_5032; Manufacturer Part Number ASFL1-24.576MHZ-EC-T -> SX5M24.576M20F30TNN; Supplier Part Numbers {"jlcpcb": ["C17566269"]} -> {"jlcpcb": ["C2901534"]}
- Y_XU: value FA-238 24.0000MD30X-W5 -> X322524MOB4SI; footprint crow_usb_digital:Epson_FA238_3225_4Pin -> crow_usb_digital:YXC_YSX321SL_3225_4Pin; Manufacturer Part Number FA-238 24.0000MD30X-W5 -> X322524MOB4SI; Supplier Part Numbers {"jlcpcb": ["C2650433"]} -> {"jlcpcb": ["C70590"]}
Connections:
- net ADC_MCLK_RAW is gone; now on net GND: U_ADC_OUT.1 (1A)
- net ADC1N: now also C_ADC_AC1N1.2, C_ADC_AC1N2.2, U_ADC_A.13 (IN4M); no longer R_ADC_PD1N.1, U_ISO1.6 (D2)
- net ADC1P: now also C_ADC_AC1P1.2, C_ADC_AC1P2.2, U_ADC_A.12 (IN4P); no longer R_ADC_PD1P.1, U_ISO1.2 (D1)
- net ADC2N: now also C_ADC_AC2N1.2, C_ADC_AC2N2.2, U_ADC_A.11 (IN3M); no longer R_ADC_PD2N.1, U_ISO2.6 (D2)
- net ADC2P: now also C_ADC_AC2P1.2, C_ADC_AC2P2.2, U_ADC_A.10 (IN3P); no longer R_ADC_PD2P.1, U_ISO2.2 (D1)
- net ADC3N: now also C_ADC_AC3N1.2, C_ADC_AC3N2.2, U_ADC_A.9 (IN2M); no longer R_ADC_PD3N.1, U_ISO3.6 (D2)
- net ADC3P: now also C_ADC_AC3P1.2, C_ADC_AC3P2.2, U_ADC_A.8 (IN2P); no longer R_ADC_PD3P.1, U_ISO3.2 (D1)
- net ADC4N: now also C_ADC_AC4N1.2, C_ADC_AC4N2.2, U_ADC_A.7 (IN1M); no longer R_ADC_PD4N.1, U_ISO4.6 (D2)
- net ADC4P: now also C_ADC_AC4P1.2, C_ADC_AC4P2.2, U_ADC_A.6 (IN1P); no longer R_ADC_PD4P.1, U_ISO4.2 (D1)
- net ADC5N: now also C_ADC_AC5N1.2, C_ADC_AC5N2.2, U_ADC_B.7 (IN1M); no longer R_ADC_PD5N.1, U_ISO5.6 (D2)
- net ADC5P: now also C_ADC_AC5P1.2, C_ADC_AC5P2.2, U_ADC_B.6 (IN1P); no longer R_ADC_PD5P.1, U_ISO5.2 (D1)
- net ADC6N: now also C_ADC_AC6N1.2, C_ADC_AC6N2.2, U_ADC_B.9 (IN2M); no longer R_ADC_PD6N.1, U_ISO6.6 (D2)
- net ADC6P: now also C_ADC_AC6P1.2, C_ADC_AC6P2.2, U_ADC_B.8 (IN2P); no longer R_ADC_PD6P.1, U_ISO6.2 (D1)
- net ADC7N: now also C_ADC_AC7N1.2, C_ADC_AC7N2.2, U_ADC_B.11 (IN3M); no longer R_ADC_PD7N.1, U_ISO7.6 (D2)
- net ADC7P: now also C_ADC_AC7P1.2, C_ADC_AC7P2.2, U_ADC_B.10 (IN3P); no longer R_ADC_PD7P.1, U_ISO7.2 (D1)
- net ADC8N: now also C_ADC_AC8N1.2, C_ADC_AC8N2.2, U_ADC_B.13 (IN4M); no longer R_ADC_PD8N.1, U_ISO8.6 (D2)
- net ADC8P: now also C_ADC_AC8P1.2, C_ADC_AC8P2.2, U_ADC_B.12 (IN4P); no longer R_ADC_PD8P.1, U_ISO8.2 (D1)
- net ADC_BCLK: now also U_ADC_A.22 (BCLK), U_ADC_B.22 (BCLK)
- net ADC_DOUT1: now also U_ADC_A.21 (SDOUT), U_ADC_B.21 (SDOUT)
- net ADC_FSYNC: now also U_ADC_A.23 (FSYNC), U_ADC_B.23 (FSYNC)
- net ADC_READY: now also U_ADC_I2C_XLATE.6 (OE)
- net ADC_RESET_N: now also Q_ADC_PWR_RST.3 (D), U_ADC_A.14 (SHDNZ), U_ADC_B.14 (SHDNZ)
- net AUDIO_EN: now also U_ISO1.2 (SEL), U_ISO2.2 (SEL), U_ISO3.2 (SEL), U_ISO4.2 (SEL), U_ISO5.2 (SEL), U_ISO6.2 (SEL), U_ISO7.2 (SEL), U_ISO8.2 (SEL); no longer U_ISO1.3 (SEL2), U_ISO1.7 (SEL1), U_ISO2.3 (SEL2), U_ISO2.7 (SEL1), U_ISO3.3 (SEL2), U_ISO3.7 (SEL1), U_ISO4.3 (SEL2), U_ISO4.7 (SEL1), U_ISO5.3 (SEL2), U_ISO5.7 (SEL1), U_ISO6.3 (SEL2), U_ISO6.7 (SEL1), U_ISO7.3 (SEL2), U_ISO7.7 (SEL1), U_ISO8.3 (SEL2), U_ISO8.7 (SEL1)
- net BUCK_AGND: now also R_BUCK_FB_BOTTOM.2
- net DUMP_RC: now also C_DUMP_TIME1.1, C_DUMP_TIME2.1, C_DUMP_TIME3.1, C_DUMP_TIME4.1, C_DUMP_TIME5.1, C_DUMP_TIME6.1, C_DUMP_TIME7.1, C_DUMP_TIME8.1, R_DUMP_TIME3.2; no longer R_DUMP_TIME1.2
- net FILTER1N: now also U_ISO1.9 (S2B); no longer U_ISO1.5 (S2)
- net FILTER1P: now also U_ISO1.7 (S1B); no longer U_ISO1.1 (S1)
- net FILTER2N: now also U_ISO2.9 (S2B); no longer U_ISO2.5 (S2)
- net FILTER2P: now also U_ISO2.7 (S1B); no longer U_ISO2.1 (S1)
- net FILTER3N: now also U_ISO3.9 (S2B); no longer U_ISO3.5 (S2)
- net FILTER3P: now also U_ISO3.7 (S1B); no longer U_ISO3.1 (S1)
- net FILTER4N: now also U_ISO4.9 (S2B); no longer U_ISO4.5 (S2)
- net FILTER4P: now also U_ISO4.7 (S1B); no longer U_ISO4.1 (S1)
- net FILTER5N: now also U_ISO5.9 (S2B); no longer U_ISO5.5 (S2)
- net FILTER5P: now also U_ISO5.7 (S1B); no longer U_ISO5.1 (S1)
- net FILTER6N: now also U_ISO6.9 (S2B); no longer U_ISO6.5 (S2)
- net FILTER6P: now also U_ISO6.7 (S1B); no longer U_ISO6.1 (S1)
- net FILTER7N: now also U_ISO7.9 (S2B); no longer U_ISO7.5 (S2)
- net FILTER7P: now also U_ISO7.7 (S1B); no longer U_ISO7.1 (S1)
- net FILTER8N: now also U_ISO8.9 (S2B); no longer U_ISO8.5 (S2)
- net FILTER8P: now also U_ISO8.7 (S1B); no longer U_ISO8.1 (S1)
- net GND: now also U_ISO1.5 (GND), U_ISO2.5 (GND), U_ISO3.5 (GND), U_ISO4.5 (GND), U_ISO5.5 (GND), U_ISO6.5 (GND), U_ISO7.5 (GND), U_ISO8.5 (GND), C_ADC_A_AREG_100N.2, C_ADC_A_AREG_1U.2, C_ADC_A_AVDD_100N.2, C_ADC_A_AVDD_10U.2, C_ADC_A_DREG_100N.2, C_ADC_A_DREG_1U.2, C_ADC_A_IOVDD_100N.2, C_ADC_A_IOVDD_10U.2, C_ADC_A_VREF_100N.2, C_ADC_A_VREF_10U.2, C_ADC_B_AREG_100N.2, C_ADC_B_AREG_1U.2, C_ADC_B_AVDD_100N.2, C_ADC_B_AVDD_10U.2, C_ADC_B_DREG_100N.2, C_ADC_B_DREG_1U.2, C_ADC_B_IOVDD_100N.2, C_ADC_B_IOVDD_10U.2, C_ADC_B_VREF_100N.2, C_ADC_B_VREF_10U.2, C_ADC_I2C_A.2, C_ADC_I2C_B.2, C_ADC_PWR_BAD.2, C_DUMP_TIME1.2, C_DUMP_TIME2.2, C_DUMP_TIME3.2, C_DUMP_TIME4.2, C_DUMP_TIME5.2, C_DUMP_TIME6.2, C_DUMP_TIME7.2, C_DUMP_TIME8.2, C_HOLD10.2, C_HOLD11.2, C_HOLD12.2, C_HOLD13.2, C_HOLD14.2, C_HOLD15.2, C_HOLD16.2, C_HOLD3.2, C_HOLD4.2, C_HOLD5.2, C_HOLD6.2, C_HOLD7.2, C_HOLD8.2, C_HOLD9.2, C_PWR_CT2.2, C_PWR_CT3.2, Q_ADC_PWR_RST.2 (S), R_1V8_FB_BOTTOM.2, R_1V8_OK_BOT.2, R_3V3X_FB_BOTTOM.2, R_ADC_1V8_OK_BOT.2, R_ADC_3V3X_OK_BOT.2, R_ADC_OK_BOT.2, R_ADC_PWR_BAD_PD.2, R_XU_3V3_OK_BOT.2, U_ADC_A.15 (ADDR1), U_ADC_A.16 (ADDR0), U_ADC_A.25 (EP_VSS), U_ADC_A.4 (AVSS), U_ADC_B.15 (ADDR1), U_ADC_B.25 (EP_VSS), U_ADC_B.4 (AVSS), U_ADC_I2C_XLATE.2 (GND), U_ADC_PWR_BAD.3 (GND); no longer U_ISO1.4 (GND), U_ISO1.9 (EP), U_ISO2.4 (GND), U_ISO2.9 (EP), U_ISO3.4 (GND), U_ISO3.9 (EP), U_ISO4.4 (GND), U_ISO4.9 (EP), U_ISO5.4 (GND), U_ISO5.9 (EP), U_ISO6.4 (GND), U_ISO6.9 (EP), U_ISO7.4 (GND), U_ISO7.9 (EP), U_ISO8.4 (GND), U_ISO8.9 (EP)
- net N0V9: now also C_CORE_FF.1
- net N1V8: now also C_1V8_FF.1, C_ADC_I2C_A.1, R_1V8_FB_TOP.1, R_1V8_OK_TOP.1, R_ADC_1V8_OK_TOP.1, R_ADC_I2C_SCL_A_PU.2, R_ADC_I2C_SDA_A_PU.2, U_ADC_I2C_XLATE.3 (VCCA); no longer U_1V8.3 (FB), U_1V8_OK.1 (SENSE), U_ADC_1V8_OK.1 (SENSE)
- net N3V3X: now also C_3V3X_FF.1, R_3V3X_FB_TOP.1, R_ADC_3V3X_OK_TOP.1, R_XU_3V3_OK_TOP.1; no longer U_3V3X.3 (FB), U_ADC_3V3X_OK.1 (SENSE), U_XU_3V3_OK.1 (SENSE)
- net N3V3_ADC: now also C_ADC_A_AVDD_100N.1, C_ADC_A_AVDD_10U.1, C_ADC_A_IOVDD_100N.1, C_ADC_A_IOVDD_10U.1, C_ADC_B_AVDD_100N.1, C_ADC_B_AVDD_10U.1, C_ADC_B_IOVDD_100N.1, C_ADC_B_IOVDD_10U.1, C_ADC_I2C_B.1, R_ADC_I2C_SCL_B_PU.2, R_ADC_I2C_SDA_B_PU.2, R_ADC_OK_TOP.1, U_ADC_A.1 (AVDD), U_ADC_A.19 (IOVDD), U_ADC_B.1 (AVDD), U_ADC_B.16 (ADDR0), U_ADC_B.19 (IOVDD), U_ADC_I2C_XLATE.7 (VCCB); no longer U_ADC_OK.1 (SENSE)
- net N5V_BUCK: now also R_BUCK_FB_TOP.1; no longer U_BUCK.25 (FB)
- net N5V_LDO_HOLD: now also C_ADC_PWR_BAD.1, C_HOLD10.1, C_HOLD11.1, C_HOLD12.1, C_HOLD13.1, C_HOLD14.1, C_HOLD15.1, C_HOLD16.1, C_HOLD3.1, C_HOLD4.1, C_HOLD5.1, C_HOLD6.1, C_HOLD7.1, C_HOLD8.1, C_HOLD9.1, U_ADC_PWR_BAD.5 (VCC)
- net PWR_CT: now also C_PWR_CT2.1, C_PWR_CT3.1
- net PWR_EN: now also U_ADC_PWR_BAD.2 (A); no longer R_DUMP_TIME2.1
- net U_CORE_FB: now also C_CORE_FF.2
- net XU_I2C_SCL_1V8: now reaches U_XU.93 (X0D35_I2C_SCL)
- net XU_I2C_SCL_1V8: now also R_ADC_I2C_SCL_A_PU.1, U_ADC_I2C_XLATE.5 (SCL_A)
- net XU_I2C_SDA_1V8: now reaches U_XU.94 (X0D36_I2C_SDA)
- net XU_I2C_SDA_1V8: now also R_ADC_I2C_SDA_A_PU.1, U_ADC_I2C_XLATE.4 (SDA_A)
- net ADC_MCLK_SAFE: no longer names the net of U_ADC_OUT.7 (1Y)
- new net ADC_A_AREG: C_ADC_A_AREG_100N.1, C_ADC_A_AREG_1U.1, U_ADC_A.2 (AREG)
- new net ADC_A_DREG: C_ADC_A_DREG_100N.1, C_ADC_A_DREG_1U.1, U_ADC_A.24 (DREG)
- new net ADC_A_VREF: C_ADC_A_VREF_100N.1, C_ADC_A_VREF_10U.1, U_ADC_A.3 (VREF)
- new net ADC_B_AREG: C_ADC_B_AREG_100N.1, C_ADC_B_AREG_1U.1, U_ADC_B.2 (AREG)
- new net ADC_B_DREG: C_ADC_B_DREG_100N.1, C_ADC_B_DREG_1U.1, U_ADC_B.24 (DREG)
- new net ADC_B_VREF: C_ADC_B_VREF_100N.1, C_ADC_B_VREF_10U.1, U_ADC_B.3 (VREF)
- new net ADC_I2C_SCL: R_ADC_I2C_SCL_B_PU.1, U_ADC_A.17 (SCL), U_ADC_B.17 (SCL), U_ADC_I2C_XLATE.8 (SCL_B)
- new net ADC_I2C_SDA: R_ADC_I2C_SDA_B_PU.1, U_ADC_A.18 (SDA), U_ADC_B.18 (SDA), U_ADC_I2C_XLATE.1 (SDA_B)
- new net ADC_PWR_BAD: Q_ADC_PWR_RST.1 (G), R_ADC_PWR_BAD_PD.1, U_ADC_PWR_BAD.4 (Y)
- new net BUCK_FB: R_BUCK_FB_BOTTOM.1, R_BUCK_FB_TOP.2, U_BUCK.25 (FB)
- new net DUMP_RMID: R_DUMP_TIME1.2, R_DUMP_TIME2.1, R_DUMP_TIME3.1
- new net ISO1N: C_ADC_AC1N1.1, C_ADC_AC1N2.1, R_ADC_PD1N.1, U_ISO1.6 (D2)
- new net ISO1P: C_ADC_AC1P1.1, C_ADC_AC1P2.1, R_ADC_PD1P.1, U_ISO1.4 (D1)
- new net ISO2N: C_ADC_AC2N1.1, C_ADC_AC2N2.1, R_ADC_PD2N.1, U_ISO2.6 (D2)
- new net ISO2P: C_ADC_AC2P1.1, C_ADC_AC2P2.1, R_ADC_PD2P.1, U_ISO2.4 (D1)
- new net ISO3N: C_ADC_AC3N1.1, C_ADC_AC3N2.1, R_ADC_PD3N.1, U_ISO3.6 (D2)
- new net ISO3P: C_ADC_AC3P1.1, C_ADC_AC3P2.1, R_ADC_PD3P.1, U_ISO3.4 (D1)
- new net ISO4N: C_ADC_AC4N1.1, C_ADC_AC4N2.1, R_ADC_PD4N.1, U_ISO4.6 (D2)
- new net ISO4P: C_ADC_AC4P1.1, C_ADC_AC4P2.1, R_ADC_PD4P.1, U_ISO4.4 (D1)
- new net ISO5N: C_ADC_AC5N1.1, C_ADC_AC5N2.1, R_ADC_PD5N.1, U_ISO5.6 (D2)
- new net ISO5P: C_ADC_AC5P1.1, C_ADC_AC5P2.1, R_ADC_PD5P.1, U_ISO5.4 (D1)
- new net ISO6N: C_ADC_AC6N1.1, C_ADC_AC6N2.1, R_ADC_PD6N.1, U_ISO6.6 (D2)
- new net ISO6P: C_ADC_AC6P1.1, C_ADC_AC6P2.1, R_ADC_PD6P.1, U_ISO6.4 (D1)
- new net ISO7N: C_ADC_AC7N1.1, C_ADC_AC7N2.1, R_ADC_PD7N.1, U_ISO7.6 (D2)
- new net ISO7P: C_ADC_AC7P1.1, C_ADC_AC7P2.1, R_ADC_PD7P.1, U_ISO7.4 (D1)
- new net ISO8N: C_ADC_AC8N1.1, C_ADC_AC8N2.1, R_ADC_PD8N.1, U_ISO8.6 (D2)
- new net ISO8P: C_ADC_AC8P1.1, C_ADC_AC8P2.1, R_ADC_PD8P.1, U_ISO8.4 (D1)
- new net U_1V8_FB: C_1V8_FF.2, R_1V8_FB_BOTTOM.1, R_1V8_FB_TOP.2, U_1V8.3 (FB)
- new net U_1V8_OK_SENSE: R_1V8_OK_BOT.1, R_1V8_OK_TOP.2, U_1V8_OK.1 (SENSE)
- new net U_3V3X_FB: C_3V3X_FF.2, R_3V3X_FB_BOTTOM.1, R_3V3X_FB_TOP.2, U_3V3X.3 (FB)
- new net U_ADC_1V8_OK_SENSE: R_ADC_1V8_OK_BOT.1, R_ADC_1V8_OK_TOP.2, U_ADC_1V8_OK.1 (SENSE)
- new net U_ADC_3V3X_OK_SENSE: R_ADC_3V3X_OK_BOT.1, R_ADC_3V3X_OK_TOP.2, U_ADC_3V3X_OK.1 (SENSE)
- new net U_ADC_OK_SENSE: R_ADC_OK_BOT.1, R_ADC_OK_TOP.2, U_ADC_OK.1 (SENSE)
- new net U_XU_3V3_OK_SENSE: R_XU_3V3_OK_BOT.1, R_XU_3V3_OK_TOP.2, U_XU_3V3_OK.1 (SENSE)
- no-connect marks 126 -> 143
Other:
- note removed: "REFERENCES"

Commit message: Accept Crow DLC USB schematic and reconcile block interfaces
Parts:
- C_U_1V8_IN_1, C_U_1V8_IN_2, C_U_3V3X_IN_1, C_U_3V3X_IN_2, C_U_CORE_IN_1, C_U_CORE_IN_2: Manufacturer Part Number CL21A106KOCLRNC -> CL21A106KOQNNNE; Supplier Part Numbers {"jlcpcb": ["C318695"]} -> {"jlcpcb": ["C1713"]}
- J_USB: value USB4105-GF-A-120 -> USB4215-03-A; footprint crow_usb_carrier_v1:GCT_USB4105_GF_A_120 -> crow_usb_carrier_v1:GCT_USB4215_03_A; Manufacturer Part Number USB4105-GF-A-120 -> USB4215-03-A; Supplier Part Numbers {"jlcpcb": ["C5184243"]} -> {"jlcpcb": ["C37616412"]}
- R_3V3X_FB_TOP: Manufacturer Part Number RT0603BRD07453KL -> ARG03BTC4533; Supplier Part Numbers {"jlcpcb": ["C861412"]} -> {"jlcpcb": ["C2686428"]}
- U_1V8, U_3V3X, U_CORE: value TPS62825DMQR -> TPS62822DLCR; footprint crow_usb_digital:TI_DMQ0006A_VSON6 -> crow_usb_digital:TI_DLC0008B_VSON_HR8; Manufacturer Part Number TPS62825DMQR -> TPS62822DLCR; Supplier Part Numbers {"jlcpcb": ["C2650334"]} -> {"jlcpcb": ["C473385"]}
Connections:
- net GND: now also J_USB.A1 (A1_GND), J_USB.A12 (A12_GND), J_USB.B1 (B1_GND), J_USB.B12 (B12_GND), J_USB.SH (SHIELD), U_1V8.3 (AGND), U_1V8.5 (PGND), U_3V3X.3 (AGND), U_3V3X.5 (PGND), U_CORE.3 (AGND), U_CORE.5 (PGND); no longer J_USB.1 (A1_GND), J_USB.16 (B12_GND), J_USB.17 (SHIELD), J_USB.8 (A12_GND), J_USB.9 (B1_GND), U_1V8.4 (GND), U_3V3X.4 (GND), U_CORE.4 (GND)
- net N5V_BUCK: now also U_1V8.7 (VIN), U_3V3X.7 (VIN), U_CORE.7 (VIN); no longer U_1V8.6 (VIN), U_3V3X.6 (VIN), U_CORE.6 (VIN)
- net USB_CC1: now also J_USB.A5 (A5_CC1); no longer J_USB.3 (A5_CC1)
- net USB_CC2: now also J_USB.B5 (B5_CC2); no longer J_USB.11 (B5_CC2)
- net USB_DN: now also J_USB.A7 (A7_DM), J_USB.B7 (B7_DM); no longer J_USB.13 (B7_DM), J_USB.5 (A7_DM)
- net USB_DP: now also J_USB.A6 (A6_DP), J_USB.B6 (B6_DP); no longer J_USB.12 (B6_DP), J_USB.4 (A6_DP)
- net U_1V8_FB: now also U_1V8.2 (FB); no longer U_1V8.3 (FB)
- net U_1V8_SW: now also U_1V8.6 (SW); no longer U_1V8.5 (SW)
- net U_3V3X_FB: now also U_3V3X.2 (FB); no longer U_3V3X.3 (FB)
- net U_3V3X_SW: now also U_3V3X.6 (SW); no longer U_3V3X.5 (SW)
- net U_CORE_FB: now also U_CORE.2 (FB); no longer U_CORE.3 (FB)
- net U_CORE_SW: now also U_CORE.6 (SW); no longer U_CORE.5 (SW)
- net VBUS_USB: now also J_USB.A4 (A4_VBUS), J_USB.A9 (A9_VBUS), J_USB.B4 (B4_VBUS), J_USB.B9 (B9_VBUS); no longer J_USB.10 (B4_VBUS), J_USB.15 (B9_VBUS), J_USB.2 (A4_VBUS), J_USB.7 (A9_VBUS)
- no-connect marks 143 -> 146

Commit message: Checkpoint Crow 45-page pre-route reviews (WIP; DO-NOT-ORDER)
Parts:
- added C_ADC_3V3X_OK_VDD: 100nF, Capacitor_SMD:C_0402_1005Metric, symbol elt:SYM_C_ADC_3V3X_OK_VDD
Connections:
- net GND: now also C_ADC_3V3X_OK_VDD.2
- net N3V3_ADC: now also C_ADC_3V3X_OK_VDD.1

Commit message: Use TI DRL land pattern for TPD2E2U06 ESD arrays
Parts:
- U_ESD1, U_ESD2, U_ESD3, U_ESD4, U_ESD5, U_ESD6, U_ESD7, U_ESD8, U_USB_CC_ESD, U_USB_VBUS_ESD: footprint Package_TO_SOT_SMD:SOT-553 -> crow_usb_analog:TI_DRL0005A_TPD2E2U06
Changed lines of the file:
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@@
     (property "Reference" "U_ESD1" (at 64.770 2121.875 0) (effects (font (size 1.27 1.27))))
     (property "Value" "TPD2E2U06DRLR" (at 64.770 2141.515 0) (effects (font (size 1.27 1.27))))
-    (property "Footprint" "Package_TO_SOT_SMD:SOT-553" (at 64.770 2127.885 0) (effects (font (size 1.27 1.27)) hide))
+    (property "Footprint" "crow_usb_analog:TI_DRL0005A_TPD2E2U06" (at 64.770 2127.885 0) (effects (font (size 1.27 1.27)) hide))
     (property "Datasheet" "https://www.ti.com/lit/ds/symlink/tpd2e2u06.pdf" (at 64.770 2127.885 0) (effects (font (size 1.27 1.27)) hide))
     (property "Manufacturer Part Number" "TPD2E2U06DRLR" (at 64.770 2127.885 0) (effects (font (size 1.27 1.27)) hide))
@@
     (property "Reference" "U_ESD2" (at 64.770 2302.215 0) (effects (font (size 1.27 1.27))))
     (property "Value" "TPD2E2U06DRLR" (at 64.770 2321.855 0) (effects (font (size 1.27 1.27))))
-    (property "Footprint" "Package_TO_SOT_SMD:SOT-553" (at 64.770 2308.225 0) (effects (font (size 1.27 1.27)) hide))
+    (property "Footprint" "crow_usb_analog:TI_DRL0005A_TPD2E2U06" (at 64.770 2308.225 0) (effects (font (size 1.27 1.27)) hide))
     (property "Datasheet" "https://www.ti.com/lit/ds/symlink/tpd2e2u06.pdf" (at 64.770 2308.225 0) (effects (font (size 1.27 1.27)) hide))
     (property "Manufacturer Part Number" "TPD2E2U06DRLR" (at 64.770 2308.225 0) (effects (font (size 1.27 1.27)) hide))
@@
     (property "Reference" "U_ESD3" (at 64.770 2482.555 0) (effects (font (size 1.27 1.27))))
     (property "Value" "TPD2E2U06DRLR" (at 64.770 2502.195 0) (effects (font (size 1.27 1.27))))
-    (property "Footprint" "Package_TO_SOT_SMD:SOT-553" (at 64.770 2488.565 0) (effects (font (size 1.27 1.27)) hide))
+    (property "Footprint" "crow_usb_analog:TI_DRL0005A_TPD2E2U06" (at 64.770 2488.565 0) (effects (font (size 1.27 1.27)) hide))
     (property "Datasheet" "https://www.ti.com/lit/ds/symlink/tpd2e2u06.pdf" (at 64.770 2488.565 0) (effects (font (size 1.27 1.27)) hide))
     (property "Manufacturer Part Number" "TPD2E2U06DRLR" (at 64.770 2488.565 0) (effects (font (size 1.27 1.27)) hide))
@@
     (property "Reference" "U_ESD4" (at 64.770 2662.895 0) (effects (font (size 1.27 1.27))))
     (property "Value" "TPD2E2U06DRLR" (at 64.770 2682.535 0) (effects (font (size 1.27 1.27))))
-    (property "Footprint" "Package_TO_SOT_SMD:SOT-553" (at 64.770 2668.905 0) (effects (font (size 1.27 1.27)) hide))
+    (property "Footprint" "crow_usb_analog:TI_DRL0005A_TPD2E2U06" (at 64.770 2668.905 0) (effects (font (size 1.27 1.27)) hide))
     (property "Datasheet" "https://www.ti.com/lit/ds/symlink/tpd2e2u06.pdf" (at 64.770 2668.905 0) (effects (font (size 1.27 1.27)) hide))
     (property "Manufacturer Part Number" "TPD2E2U06DRLR" (at 64.770 2668.905 0) (effects (font (size 1.27 1.27)) hide))
@@
     (property "Reference" "U_ESD5" (at 64.770 2843.235 0) (effects (font (size 1.27 1.27))))
     (property "Value" "TPD2E2U06DRLR" (at 64.770 2862.875 0) (effects (font (size 1.27 1.27))))
-    (property "Footprint" "Package_TO_SOT_SMD:SOT-553" (at 64.770 2849.245 0) (effects (font (size 1.27 1.27)) hide))
+    (property "Footprint" "crow_usb_analog:TI_DRL0005A_TPD2E2U06" (at 64.770 2849.245 0) (effects (font (size 1.27 1.27)) hide))
     (property "Datasheet" "https://www.ti.com/lit/ds/symlink/tpd2e2u06.pdf" (at 64.770 2849.245 0) (effects (font (size 1.27 1.27)) hide))
     (property "Manufacturer Part Number" "TPD2E2U06DRLR" (at 64.770 2849.245 0) (effects (font (size 1.27 1.27)) hide))
@@
     (property "Reference" "U_ESD6" (at 543.560 137.500 0) (effects (font (size 1.27 1.27))))
     (property "Value" "TPD2E2U06DRLR" (at 543.560 157.140 0) (effects (font (size 1.27 1.27))))
-    (property "Footprint" "Package_TO_SOT_SMD:SOT-553" (at 543.560 143.510 0) (effects (font (size 1.27 1.27)) hide))
+    (property "Footprint" "crow_usb_analog:TI_DRL0005A_TPD2E2U06" (at 543.560 143.510 0) (effects (font (size 1.27 1.27)) hide))
     (property "Datasheet" "https://www.ti.com/lit/ds/symlink/tpd2e2u06.pdf" (at 543.560 143.510 0) (effects (font (size 1.27 1.27)) hide))
     (property "Manufacturer Part Number" "TPD2E2U06DRLR" (at 543.560 143.510 0) (effects (font (size 1.27 1.27)) hide))
@@
     (property "Reference" "U_ESD7" (at 543.560 317.840 0) (effects (font (size 1.27 1.27))))
     (property "Value" "TPD2E2U06DRLR" (at 543.560 337.480 0) (effects (font (size 1.27 1.27))))
-    (property "Footprint" "Package_TO_SOT_SMD:SOT-553" (at 543.560 323.850 0) (effects (font (size 1.27 1.27)) hide))
+    (property "Footprint" "crow_usb_analog:TI_DRL0005A_TPD2E2U06" (at 543.560 323.850 0) (effects (font (size 1.27 1.27)) hide))
     (property "Datasheet" "https://www.ti.com/lit/ds/symlink/tpd2e2u06.pdf" (at 543.560 323.850 0) (effects (font (size 1.27 1.27)) hide))
     (property "Manufacturer Part Number" "TPD2E2U06DRLR" (at 543.560 323.850 0) (effects (font (size 1.27 1.27)) hide))
@@
     (property "Reference" "U_ESD8" (at 543.560 498.815 0) (effects (font (size 1.27 1.27))))
     (property "Value" "TPD2E2U06DRLR" (at 543.560 518.455 0) (effects (font (size 1.27 1.27))))
-    (property "Footprint" "Package_TO_SOT_SMD:SOT-553" (at 543.560 504.825 0) (effects (font (size 1.27 1.27)) hide))
+    (property "Footprint" "crow_usb_analog:TI_DRL0005A_TPD2E2U06" (at 543.560 504.825 0) (effects (font (size 1.27 1.27)) hide))
     (property "Datasheet" "https://www.ti.com/lit/ds/symlink/tpd2e2u06.pdf" (at 543.560 504.825 0) (effects (font (size 1.27 1.27)) hide))
     (property "Manufacturer Part Number" "TPD2E2U06DRLR" (at 543.560 504.825 0) (effects (font (size 1.27 1.27)) hide))
@@
     (property "Reference" "U_USB_CC_ESD" (at 1286.510 930.615 0) (effects (font (size 1.27 1.27))))
     (property "Value" "TPD2E2U06DRLR" (at 1286.510 945.175 0) (effects (font (size 1.27 1.27))))
-    (property "Footprint" "Package_TO_SOT_SMD:SOT-553" (at 1286.510 937.895 0) (effects (font (size 1.27 1.27)) hide))
+    (property "Footprint" "crow_usb_analog:TI_DRL0005A_TPD2E2U06" (at 1286.510 937.895 0) (effects (font (size 1.27 1.27)) hide))
     (property "Datasheet" "https://www.ti.com/lit/ds/symlink/tpd2e2u06.pdf" (at 1286.510 937.895 0) (effects (font (size 1.27 1.27)) hide))
     (property "Manufacturer Part Number" "TPD2E2U06DRLR" (at 1286.510 937.895 0) (effects (font (size 1.27 1.27)) hide))
@@
     (property "Reference" "U_USB_VBUS_ESD" (at 1286.510 790.915 0) (effects (font (size 1.27 1.27))))
     (property "Value" "TPD2E2U06DRLR" (at 1286.510 805.475 0) (effects (font (size 1.27 1.27))))
-    (property "Footprint" "Package_TO_SOT_SMD:SOT-553" (at 1286.510 798.195 0) (effects (font (size 1.27 1.27)) hide))
+    (property "Footprint" "crow_usb_analog:TI_DRL0005A_TPD2E2U06" (at 1286.510 798.195 0) (effects (font (size 1.27 1.27)) hide))
     (property "Datasheet" "https://www.ti.com/lit/ds/symlink/tpd2e2u06.pdf" (at 1286.510 798.195 0) (effects (font (size 1.27 1.27)) hide))
     (property "Manufacturer Part Number" "TPD2E2U06DRLR" (at 1286.510 798.195 0) (effects (font (size 1.27 1.27)) hide))
